File: robot001.brd (EAGLE design)
At the start: 61 x 70 mm, 54 parts, among them CN1 PMX42_56579-0576, U1 ESP32-WROOM-32D, U2 LD1117S33TR, U3 DRV8833PW, U4 QRE1113GR, U5 QRE1113GR, U6 QRE1113GR, U7 QRE1113GR

Commit message: Add files via upload
Parts:
- added D1: 7.5V, SparkFun-DiscreteSemi:SOD-323
- added R16, R17: 10k, resistor:R0402
Connections:
- net +3V3: now also R16.1, R17.1
- net GND: now also D1.A
- net SCL: now also R17.2
- net SDA: now also R16.2
- net VBAT: now also D1.C
Routing:
- net +3V3: track 220.2 -> 225.5 mm
- net SDA: track 43.3 -> 48.2 mm
- net VBAT: track 6.90 -> 9.86 mm
- net SCL: track 44.7 -> 47.5 mm

Commit message: Add files via upload
Parts:
- added R18, R19: 10k, resistor:R0402
- moved R7 0.52 mm to (30.7, 30.4)
Connections:
- new net N$10: R19.2, U3.6
- new net N$9: R18.2, U3.3
- net GND: now also R18.1, R19.1
Routing:
- net N$9: track 0.00 -> 11.5 mm, vias 0 -> 2
- net N$10: track 0.00 -> 9.09 mm
Changed lines of the file:
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@@
 <attribute name="VALUE" x="39.497" y="10.033" size="0.6096" layer="27" font="vector" ratio="20" rot="R90"/>
 </element>
-<element name="R7" library="resistor" library_urn="urn:adsk.eagle:library:348" package="R0402" package3d_urn="urn:adsk.eagle:package:26058/2" value="100" x="31.215" y="30.21" smashed="yes" rot="R180">
-<attribute name="NAME" x="32.231" y="29.575" size="0.6096" layer="25" rot="R180"/>
-<attribute name="VALUE" x="31.85" y="32.115" size="1.27" layer="27" rot="R180"/>
+<element name="R7" library="resistor" library_urn="urn:adsk.eagle:library:348" package="R0402" package3d_urn="urn:adsk.eagle:package:26058/2" value="100" x="30.715" y="30.36" smashed="yes" rot="R180">
+<attribute name="NAME" x="31.731" y="29.725" size="0.6096" layer="25" rot="R180"/>
+<attribute name="VALUE" x="31.35" y="32.265" size="1.27" layer="27" rot="R180"/>
 </element>
 <element name="C3" library="resistor" library_urn="urn:adsk.eagle:library:348" package="C0402" package3d_urn="urn:adsk.eagle:package:23626/2" value="2.2uf" x="23.622" y="32.766" smashed="yes" rot="R180">
@@
 <attribute name="NAME" x="31.285" y="60.815" size="0.6096" layer="25" rot="R180"/>
 <attribute name="VALUE" x="31.735" y="61.505" size="1.27" layer="27" rot="R180"/>
+</element>
+<element name="R18" library="resistor" library_urn="urn:adsk.eagle:library:348" package="R0402" package3d_urn="urn:adsk.eagle:package:26058/2" value="10k" x="31.8" y="26.55" smashed="yes">
+<attribute name="NAME" x="31.165" y="25.285" size="0.6096" layer="25"/>
+<attribute name="VALUE" x="31.165" y="24.645" size="1.27" layer="27"/>
+</element>
+<element name="R19" library="resistor" library_urn="urn:adsk.eagle:library:348" package="R0402" package3d_urn="urn:adsk.eagle:package:26058/2" value="10k" x="30.8" y="27.9" smashed="yes">
+<attribute name="NAME" x="30.265" y="28.535" size="0.6096" layer="25"/>
+<attribute name="VALUE" x="30.165" y="25.995" size="1.27" layer="27"/>
 </element>
 </elements>
@@
 <contactref element="LINE_SENSOR1" pad="1"/>
 <contactref element="D1" pad="A"/>
+<contactref element="R18" pad="1"/>
+<contactref element="R19" pad="1"/>
 <wire x1="-3.55" y1="41.35" x2="2.667" y2="41.402" width="0" layer="19" extent="1-1"/>
 </signal>
@@
 <wire x1="5.207" y1="29.464" x2="5.588" y2="29.083" width="1.27" layer="16"/>
 <wire x1="5.207" y1="42.545" x2="5.207" y2="29.464" width="1.27" layer="16"/>
-<wire x1="30.565" y1="30.21" x2="29.4525" y2="29.0975" width="0.3048" layer="1"/>
+<wire x1="30.065" y1="30.36" x2="29.4525" y2="29.7475" width="0.3048" layer="1"/>
+<wire x1="29.4525" y1="29.7475" x2="29.4525" y2="29.0975" width="0.3048" layer="1"/>
 <wire x1="29.4525" y1="29.0975" x2="25.642" y2="25.287" width="0.3048" layer="1"/>
 <wire x1="25.642" y1="25.287" x2="25.642" y2="20.983" width="0.3048" layer="1"/>
@@
 <contactref element="U3" pad="1"/>
 <contactref element="R7" pad="1"/>
-<wire x1="31.865" y1="30.21" x2="32.46" y2="30.21" width="0.3048" layer="1"/>
+<wire x1="31.365" y1="30.36" x2="32.61" y2="30.36" width="0.3048" layer="1"/>
 <wire x1="33.0454" y1="30.7954" x2="33.0454" y2="31.761" width="0.3048" layer="1"/>
-<wire x1="32.46" y1="30.21" x2="33.0454" y2="30.7954" width="0.3048" layer="1"/>
+<wire x1="32.61" y1="30.36" x2="33.0454" y2="30.7954" width="0.3048" layer="1"/>
 </signal>
 <signal name="AOUT1">
@@
 <wire x1="-12.1" y1="59.1" x2="-12.1" y2="62.825" width="0.3048" layer="16"/>
 </signal>
+<signal name="N$9">
+<contactref element="U3" pad="3"/>
+<contactref element="R18" pad="2"/>
+<wire x1="32.45" y1="26.55" x2="32.45" y2="26.65393125" width="0.254" layer="1"/>
+<wire x1="32.45" y1="26.55" x2="33.25" y2="27.35" width="0.254" layer="1"/>
+<wire x1="33.25" y1="27.35" x2="34.05" y2="27.35" width="0.254" layer="1"/>
+<via x="34.05" y="27.35" extent="1-16" drill="0.35"/>
+<wire x1="34.05" y1="27.35" x2="34.05" y2="31.45" width="0.254" layer="16"/>
+<wire x1="34.05" y1="31.45" x2="33" y2="32.5" width="0.254" layer="16"/>
+<wire x1="32.95" y1="32.5" x2="33" y2="32.5" width="0.254" layer="16"/>
+<wire x1="33" y1="32.5" x2="32.5" y2="32" width="0.254" layer="16"/>
+<wire x1="32.5" y1="32" x2="31.55" y2="32" width="0.254" layer="16"/>
+<via x="31.55" y="32" extent="1-16" drill="0.35"/>
+<wire x1="31.55" y1="32" x2="31.55" y2="32.45" width="0.254" layer="1"/>
+<wire x1="32.161" y1="33.061" x2="33.0454" y2="33.061" width="0.254" layer="1"/>
+<wire x1="31.55" y1="32.45" x2="32.161" y2="33.061" width="0.254" layer="1"/>
+</signal>
+<signal name="N$10">
+<contactref element="U3" pad="6"/>
+<contactref element="R19" pad="2"/>
+<wire x1="31.45" y1="27.9" x2="31.45" y2="28.7" width="0.254" layer="1"/>
+<wire x1="31.45" y1="28.7" x2="30.7356" y2="29.4144" width="0.254" layer="1"/>
+<wire x1="31.5" y1="33" x2="31.5" y2="34.7" width="0.254" layer="1"/>
+<wire x1="31.5" y1="34.7" x2="31.811" y2="35.011" width="0.254" layer="1"/>
+<wire x1="31.811" y1="35.011" x2="33.0454" y2="35.011" width="0.254" layer="1"/>
+<wire x1="30.7356" y1="29.4144" x2="30.7356" y2="32.2356" width="0.254" layer="1"/>
+<wire x1="30.7356" y1="32.2356" x2="31.5" y2="33" width="0.254" layer="1"/>
+</signal>
 </signals>
