File: robot001.sch (EAGLE design)
At the start: 54 parts, among them CN1 PMX42_56579-0576, U1 ESP32-WROOM-32D, U2 LD1117S33TR, U3 DRV8833PW, U4 QRE1113GR, U5 QRE1113GR, U6 QRE1113GR, U7 QRE1113GR

Commit message: Add files via upload
Other:
- note removed: "mkae sure to add thsi cap to your boom"
Changed lines of the file:
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@@
 <text x="185.42" y="162.56" size="2.54" layer="94">SERVO MOTOR</text>
 <text x="7.62" y="83.82" size="2.54" layer="94">POWER</text>
-<text x="152.4" y="111.76" size="1.778" layer="94" rot="R90">mkae sure to add thsi cap to your boom</text>
-<text x="154.94" y="111.76" size="1.778" layer="94" rot="R90">mkae sure to add thsi cap to your boom</text>
-<text x="157.48" y="111.76" size="1.778" layer="94" rot="R90">mkae sure to add thsi cap to your boom</text>
-<text x="160.02" y="111.76" size="1.778" layer="94" rot="R90">mkae sure to add thsi cap to your boom</text>
-<text x="162.56" y="111.76" size="1.778" layer="94" rot="R90">mkae sure to add thsi cap to your boom</text>
 </plain>
 <instances>

Commit message: Add files via upload
Parts:
- added D1: 7.5V, SparkFun-DiscreteSemi:DIODE-ZENER-BZT52C3V6S
- added R16, R17: 10k, resistor:R-US_R0402
Connections:
- net +3V3: now also R16.1, R17.1
- net GND: now also D1.A
- net SCL: now also R17.2
- net SDA: now also R16.2
- net VBAT: now also D1.C
Changed lines of the file:
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@@
 <part name="LOGO1" library="Particle-Devices" library_urn="urn:adsk.eagle:library:5952892" deviceset="OSHW-LOGO" device="S" package3d_urn="urn:adsk.eagle:package:5952927/1"/>
 <part name="FRAME4" library="frames" library_urn="urn:adsk.eagle:library:229" deviceset="A4L-LOC" device=""/>
+<part name="D1" library="SparkFun-DiscreteSemi" library_urn="urn:adsk.eagle:library:514" deviceset="DIODE-ZENER" device="-BZT52C3V6S" package3d_urn="urn:adsk.eagle:package:38441/1" value="7.5V"/>
+<part name="GND28" library="supply1" library_urn="urn:adsk.eagle:library:371" deviceset="GND" device=""/>
+<part name="R16" library="resistor" library_urn="urn:adsk.eagle:library:348" deviceset="R-US_" device="R0402" package3d_urn="urn:adsk.eagle:package:26058/2" value="10k"/>
+<part name="R17" library="resistor" library_urn="urn:adsk.eagle:library:348" deviceset="R-US_" device="R0402" package3d_urn="urn:adsk.eagle:package:26058/2" value="10k"/>
+<part name="+3V21" library="supply1" library_urn="urn:adsk.eagle:library:371" deviceset="+3V3" device=""/>
 </parts>
 <sheets>
@@
 <attribute name="SHEET" x="278.765" y="58.42" size="2.54" layer="94"/>
 </instance>
+<instance part="R16" gate="G$1" x="231.14" y="116.84" smashed="yes">
+<attribute name="NAME" x="227.33" y="118.3386" size="1.778" layer="95"/>
+<attribute name="VALUE" x="227.33" y="113.538" size="1.778" layer="96"/>
+</instance>
+<instance part="R17" gate="G$1" x="231.14" y="106.68" smashed="yes">
+<attribute name="NAME" x="227.33" y="108.1786" size="1.778" layer="95"/>
+<attribute name="VALUE" x="227.33" y="103.378" size="1.778" layer="96"/>
+</instance>
+<instance part="+3V21" gate="G$1" x="218.44" y="124.46" smashed="yes">
+<attribute name="VALUE" x="215.9" y="119.38" size="1.778" layer="96" rot="R90"/>
+</instance>
 </instances>
 <busses>
@@
 <segment>
 <pinref part="U1" gate="G$1" pin="IO26"/>
-<wire x1="132.08" y1="157.48" x2="144.78" y2="157.48" width="0.1524" layer="91"/>
-<label x="142.24" y="157.48" size="1.778" layer="95" align="bottom-right"/>
+<wire x1="132.08" y1="157.48" x2="154.94" y2="157.48" width="0.1524" layer="91"/>
+<label x="152.4" y="157.48" size="1.778" layer="95" align="bottom-right"/>
 </segment>
 </net>
@@
 <segment>
 <pinref part="U1" gate="G$1" pin="IO27"/>
-<wire x1="132.08" y1="154.94" x2="144.78" y2="154.94" width="0.1524" layer="91"/>
-<label x="142.24" y="154.94" size="1.778" layer="95" align="bottom-right"/>
+<wire x1="132.08" y1="154.94" x2="154.94" y2="154.94" width="0.1524" layer="91"/>
+<label x="152.4" y="154.94" size="1.778" layer="95" align="bottom-right"/>
 </segment>
 </net>
@@
 <pinref part="R2" gate="G$1" pin="2"/>
 <wire x1="233.68" y1="185.42" x2="236.22" y2="185.42" width="0.1524" layer="91"/>
+</segment>
+<segment>
+<pinref part="R16" gate="G$1" pin="1"/>
+<wire x1="226.06" y1="116.84" x2="218.44" y2="116.84" width="0.1524" layer="91"/>
+<wire x1="218.44" y1="116.84" x2="218.44" y2="106.68" width="0.1524" layer="91"/>
+<pinref part="R17" gate="G$1" pin="1"/>
+<wire x1="218.44" y1="106.68" x2="226.06" y2="106.68" width="0.1524" layer="91"/>
+<pinref part="+3V21" gate="G$1" pin="+3V3"/>
+<wire x1="218.44" y1="121.92" x2="218.44" y2="116.84" width="0.1524" layer="91"/>
+<junction x="218.44" y="116.84"/>
 </segment>
 </net>
@@
 <label x="154.94" y="167.64" size="1.778" layer="95" align="bottom-right"/>
 </segment>
+<segment>
+<pinref part="R16" gate="G$1" pin="2"/>
+<wire x1="236.22" y1="116.84" x2="248.92" y2="116.84" width="0.1524" layer="91"/>
+<label x="243.84" y="116.84" size="1.778" layer="95"/>
+</segment>
 </net>
 <net name="SCL" class="0">
@@
 <label x="154.94" y="165.1" size="1.778" layer="95" align="bottom-right"/>
 </segment>
+<segment>
+<pinref part="R17" gate="G$1" pin="2"/>
+<wire x1="236.22" y1="106.68" x2="248.92" y2="106.68" width="0.1524" layer="91"/>
+<label x="243.84" y="106.68" size="1.778" layer="95"/>
+</segment>
 </net>
 <net name="N$4" class="0">
@@
 <segment>
 <pinref part="U1" gate="G$1" pin="IO19"/>
-<wire x1="132.08" y1="170.18" x2="144.78" y2="170.18" width="0.1524" layer="91"/>
-<label x="142.24" y="170.18" size="1.778" layer="95" align="bottom-right"/>
+<wire x1="132.08" y1="170.18" x2="154.94" y2="170.18" width="0.1524" layer="91"/>
+<label x="152.4" y="170.18" size="1.778" layer="95" align="bottom-right"/>
 </segment>
 </net>
@@
 <segment>
 <pinref part="U1" gate="G$1" pin="IO25"/>
-<wire x1="132.08" y1="160.02" x2="144.78" y2="160.02" width="0.1524" layer="91"/>
-<label x="142.24" y="160.02" size="1.778" layer="95" align="bottom-right"/>
+<wire x1="132.08" y1="160.02" x2="154.94" y2="160.02" width="0.1524" layer="91"/>
+<label x="152.4" y="160.02" size="1.778" layer="95" align="bottom-right"/>
 </segment>
 </net>
@@
 <attribute name="VALUE" x="226.06" y="33.02" size="1.778" layer="96"/>
 </instance>
+<instance part="D1" gate="G$1" x="22.86" y="20.32" smashed="yes" rot="R90">
+<attribute name="NAME" x="20.828" y="17.78" size="1.778" layer="95" font="vector" rot="R90"/>
+<attribute name="VALUE" x="24.892" y="17.78" size="1.778" layer="96" font="vector" rot="R90" align="top-left"/>
+</instance>
+<instance part="GND28" gate="1" x="22.86" y="7.62" smashed="yes">
+<attribute name="VALUE" x="20.32" y="5.08" size="1.778" layer="96"/>
+</instance>
 </instances>
 <busses>
@@
 <wire x1="236.22" y1="38.1" x2="236.22" y2="40.64" width="0.1524" layer="91"/>
 <wire x1="236.22" y1="40.64" x2="238.76" y2="40.64" width="0.1524" layer="91"/>
+</segment>
+<segment>
+<pinref part="D1" gate="G$1" pin="A"/>
+<wire x1="22.86" y1="17.78" x2="22.86" y2="10.16" width="0.1524" layer="91"/>
+<pinref part="GND28" gate="1" pin="GND"/>
 </segment>
 </net>
@@
 <label x="96.52" y="12.7" size="1.778" layer="95"/>
 </segment>
-</net>
+<segment>
+<pinref part="D1" gate="G$1" pin="C"/>
+<wire x1="22.86" y1="22.86" x2="22.86" y2="33.02" width="0.1524" layer="91"/>
+<label x="22.86" y="27.94" size="1.778" layer="95" rot="R90"/>
+</segment>
+</net>

Commit message: Add files via upload
Parts:
- added R18, R19: 10k, resistor:R-US_R0402
Connections:
- new net N$10: R19.2, U3.BISEN
- new net N$9: R18.2, U3.AISEN
- net GND: now also R18.1, R19.1
Changed lines of the file:
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@@
 <part name="R17" library="resistor" library_urn="urn:adsk.eagle:library:348" deviceset="R-US_" device="R0402" package3d_urn="urn:adsk.eagle:package:26058/2" value="10k"/>
 <part name="+3V21" library="supply1" library_urn="urn:adsk.eagle:library:371" deviceset="+3V3" device=""/>
+<part name="R18" library="resistor" library_urn="urn:adsk.eagle:library:348" deviceset="R-US_" device="R0402" package3d_urn="urn:adsk.eagle:package:26058/2" value="10k"/>
+<part name="R19" library="resistor" library_urn="urn:adsk.eagle:library:348" deviceset="R-US_" device="R0402" package3d_urn="urn:adsk.eagle:package:26058/2" value="10k"/>
+<part name="GND29" library="supply1" library_urn="urn:adsk.eagle:library:371" deviceset="GND" device=""/>
 </parts>
 <sheets>
@@
 <attribute name="VALUE" x="20.32" y="5.08" size="1.778" layer="96"/>
 </instance>
+<instance part="R18" gate="G$1" x="35.56" y="142.24" smashed="yes">
+<attribute name="NAME" x="31.75" y="143.7386" size="1.778" layer="95"/>
+<attribute name="VALUE" x="31.75" y="138.938" size="1.778" layer="96"/>
+</instance>
+<instance part="R19" gate="G$1" x="35.56" y="134.62" smashed="yes">
+<attribute name="NAME" x="31.75" y="136.1186" size="1.778" layer="95"/>
+<attribute name="VALUE" x="31.75" y="131.318" size="1.778" layer="96"/>
+</instance>
+<instance part="GND29" gate="1" x="20.32" y="157.48" smashed="yes" rot="R180">
+<attribute name="VALUE" x="22.86" y="160.02" size="1.778" layer="96" rot="R180"/>
+</instance>
 </instances>
 <busses>
@@
 <wire x1="22.86" y1="17.78" x2="22.86" y2="10.16" width="0.1524" layer="91"/>
 <pinref part="GND28" gate="1" pin="GND"/>
+</segment>
+<segment>
+<pinref part="R18" gate="G$1" pin="1"/>
+<pinref part="GND29" gate="1" pin="GND"/>
+<wire x1="30.48" y1="142.24" x2="20.32" y2="142.24" width="0.1524" layer="91"/>
+<wire x1="20.32" y1="142.24" x2="20.32" y2="154.94" width="0.1524" layer="91"/>
+<pinref part="R19" gate="G$1" pin="1"/>
+<wire x1="30.48" y1="134.62" x2="20.32" y2="134.62" width="0.1524" layer="91"/>
+<wire x1="20.32" y1="134.62" x2="20.32" y2="142.24" width="0.1524" layer="91"/>
+<junction x="20.32" y="142.24"/>
 </segment>
 </net>
@@
 </segment>
 </net>
+<net name="N$9" class="0">
+<segment>
+<pinref part="U3" gate="A" pin="AISEN"/>
+<pinref part="R18" gate="G$1" pin="2"/>
+<wire x1="63.5" y1="142.24" x2="40.64" y2="142.24" width="0.1524" layer="91"/>
+</segment>
+</net>
+<net name="N$10" class="0">
+<segment>
+<pinref part="U3" gate="A" pin="BISEN"/>
+<pinref part="R19" gate="G$1" pin="2"/>
+<wire x1="63.5" y1="134.62" x2="40.64" y2="134.62" width="0.1524" layer="91"/>
+</segment>
+</net>
